File: clock.kicad_sch (KiCad schematic)
At the start: 40 parts, among them Q1 AOTF10N60, U1 K155NA1, U2 MAX1771xSA, U3 DS3231M, U4 TLP627, U5 TLP627, U6 TLP627, U7 TLP627

Commit message: more testing, pcb initial thing
Parts:
- added R11, R12, R13: 330, Resistor_THT:R_Axial_DIN0207_L6.3mm_D2.5mm_P10.16mm_Horizontal, symbol Device:R
- A1: footprint Module:RaspberryPi_Pico_W_SMD_HandSolder -> Module:RaspberryPi_Pico_Common_THT
- C1, C2, C4: footprint (none) -> Capacitor_THT:C_Disc_D5.0mm_W2.5mm_P2.50mm
- C3: renamed from C5; footprint (none) -> Capacitor_THT:CP_Radial_D6.3mm_P2.50mm
- C5: renamed from C3; footprint (none) -> Capacitor_THT:CP_Radial_D10.0mm_P5.00mm
- D1: footprint Package_DFN_QFN:WQFN-28-1EP_4x4mm_P0.4mm_EP2.7x2.7mm -> Diode_THT:D_DO-41_SOD81_P10.16mm_Horizontal
- D2: renamed from D3; footprint (none) -> LED_THT:LED_D3.0mm
- D3: renamed from D4; footprint (none) -> LED_THT:LED_D3.0mm
- D4: renamed from D5; footprint (none) -> LED_THT:LED_D3.0mm
- D5: renamed from D2; footprint Display_7Segment:D1X8K -> Diode_THT:D_DO-41_SOD81_P10.16mm_Horizontal
- L1: footprint (none) -> Inductor_THT:L_Radial_D10.0mm_P5.00mm_Fastron_07M
- N1, N2, N3, N4: footprint nixies-us_IN-14 -> nixies-us:nixies-us-IN-14
- Q1: footprint Package_QFP:TQFP-44_10x10mm_P0.8mm -> Package_TO_SOT_THT:TO-220-3_Vertical
- R1: renamed from R7; footprint (none) -> Resistor_THT:R_Axial_DIN0207_L6.3mm_D2.5mm_P10.16mm_Horizontal
- R10: renamed from R17; footprint (none) -> Resistor_THT:R_Axial_DIN0207_L6.3mm_D2.5mm_P10.16mm_Horizontal
- R14: renamed from R5; footprint (none) -> Resistor_THT:R_Axial_DIN0207_L6.3mm_D2.5mm_P10.16mm_Horizontal
- R15: renamed from R6; footprint (none) -> Resistor_THT:R_Axial_DIN0207_L6.3mm_D2.5mm_P10.16mm_Horizontal
- R16: renamed from R4; footprint (none) -> Resistor_THT:R_Axial_DIN0414_L11.9mm_D4.5mm_P15.24mm_Horizontal
- R17: renamed from R11; footprint (none) -> Resistor_THT:R_Axial_DIN0309_L9.0mm_D3.2mm_P12.70mm_Horizontal
- R18: renamed from R3; footprint (none) -> Resistor_THT:R_Axial_DIN0207_L6.3mm_D2.5mm_P10.16mm_Horizontal
- R2: renamed from R8; footprint (none) -> Resistor_THT:R_Axial_DIN0207_L6.3mm_D2.5mm_P10.16mm_Horizontal
- R3: renamed from R9; footprint (none) -> Resistor_THT:R_Axial_DIN0207_L6.3mm_D2.5mm_P10.16mm_Horizontal
- R4: renamed from R10; footprint (none) -> Resistor_THT:R_Axial_DIN0207_L6.3mm_D2.5mm_P10.16mm_Horizontal
- R5: renamed from R2; footprint (none) -> Resistor_THT:R_Axial_DIN0207_L6.3mm_D2.5mm_P10.16mm_Horizontal
- R6: renamed from R1; footprint (none) -> Resistor_THT:R_Axial_DIN0207_L6.3mm_D2.5mm_P10.16mm_Horizontal
- R7: renamed from R14; footprint (none) -> Resistor_THT:R_Axial_DIN0207_L6.3mm_D2.5mm_P10.16mm_Horizontal
- R8: renamed from R15; footprint (none) -> Resistor_THT:R_Axial_DIN0207_L6.3mm_D2.5mm_P10.16mm_Horizontal
- R9: renamed from R16; footprint (none) -> Resistor_THT:R_Axial_DIN0207_L6.3mm_D2.5mm_P10.16mm_Horizontal
- RV1: footprint (none) -> Potentiometer_THT:Potentiometer_Bourns_3386P_Vertical
- U1: renamed from U3; footprint Package_SO:SOIC-16W_7.5x10.3mm_P1.27mm -> Connector_PinHeader_2.54mm:PinHeader_1x04_P2.54mm_Vertical
- U6: renamed from U1; footprint Module:RaspberryPi_Pico_W_SMD_HandSolder -> Package_DIP:DIP-4_W7.62mm
- renumbered U4 to U2, U5 to U3, U6 to U4, U7 to U5, U2 to U7
Connections:
- net rtc_3v3: now reaches A1.36 (3V3), C1.1, R5.1, R6.1, U1.2 (VCC)
- net at A1.24 (GPIO18): now also R13.1; no longer D4.2 (A)
- net at Q1.1 (G), R18.1, U7.1 (EXT): now also Q1.3 (S), R16.1, U7.8 (CS)
- net at D2.2 (A): now also R11.1; no longer A1.21 (GPIO16)
- net at D3.2 (A): now also R12.1; no longer A1.22 (GPIO17)
- new net: D4.2 (A), R13.2
- new net: A1.22 (GPIO17), R12.2
- new net: A1.21 (GPIO16), R11.2
Other:
- moved on the sheet: C1, D1, D2, D3, D4, Q1, R14, R15, R5, R6, RV1, U1

Commit message: i hate pcb design
Parts:
- U6: footprint Package_DIP:DIP-4_W7.62mm -> Package_DIP:DIP-16_W7.62mm
Changed lines of the file:
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@@
 			)
 		)
-		(property "Footprint" "Package_DIP:DIP-4_W7.62mm"
+		(property "Footprint" "Package_DIP:DIP-16_W7.62mm"
 			(at 124.46 140.97 0)
 			(hide yes)
