File: clock.kicad_pcb (KiCad board)
At the start: 2 copper layers, 43 parts, among them Q1 AOTF10N60, U1 DS3231M, U2 TLP627, U3 TLP627, U4 TLP627, U5 TLP627, U6 K155NA1, U7 MAX1771xSA

Commit message: i hate pcb design
Parts:
- moved D2 132.8 mm to (280.0, 88.5), turned to 180 degrees
- moved D3 125.8 mm to (280.0, 83.0), turned to 180 degrees
- moved U2 120.8 mm to (199.8, 108.2), turned to -90 degrees
- moved U6 120.3 mm to (247.9, 100.5), turned to 0 degrees
- moved D4 119.0 mm to (280.0, 77.6), turned to 180 degrees
- moved R11 114.5 mm to (265.8, 88.2), turned to 180 degrees
- moved R10 113.9 mm to (236.6, 133.0)
- moved R8 113.9 mm to (228.4, 133.0)
- moved R9 113.9 mm to (232.5, 133.0)
- moved R12 109.5 mm to (265.8, 84.1), turned to 180 degrees
- moved R13 104.6 mm to (265.8, 80.1), turned to 180 degrees
- moved A1 104.4 mm to (231.0, 39.0), turned to 0 degrees
- moved U1 96.3 mm to (267.0, 50.2), turned to 0 degrees
- moved R7 95.8 mm to (198.0, 133.1)
- moved R1 93.1 mm to (203.0, 87.8), turned to -90 degrees
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
Commit message: more pcb layout editing...
Parts:
- U6: footprint Package_DIP:DIP-4_W7.62mm -> Package_DIP:DIP-16_W7.62mm
- moved U5 152.7 mm to (267.8, 132.7), turned to -90 degrees
- moved U4 131.6 mm to (248.5, 132.5), turned to -90 degrees
- moved R4 123.0 mm to (266.0, 110.9), turned to -90 degrees
- moved D1 108.8 mm to (266.5, 20.0), turned to 0 degrees
- moved U3 105.8 mm to (224.0, 132.5), turned to -90 degrees
- moved R3 104.5 mm to (247.0, 111.5), turned to -90 degrees
- moved R2 81.1 mm to (223.5, 113.0), turned to -90 degrees
- moved D5 42.6 mm to (135.0, 69.6)
- moved C3 39.9 mm to (143.0, 48.5), turned to 180 degrees
- moved R14 37.3 mm to (158.5, 93.5), turned to 180 degrees
- moved R10 37.2 mm to (265.0, 157.0)
- moved R15 37.0 mm to (163.9, 93.5), turned to 0 degrees
- moved R17 37.0 mm to (123.5, 58.1), turned to -90 degrees
- moved C5 34.9 mm to (151.6, 69.5), turned to 0 degrees
- moved C1 30.8 mm to (185.5, 66.0)
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
Commit message: i think it starts making sense
Parts:
- moved C1 93.5 mm to (278.5, 56.8), turned to -90 degrees
- moved D2 87.1 mm to (283.5, 1.50), turned to -90 degrees
- moved D3 81.6 mm to (278.0, 1.50), turned to -90 degrees
- moved C2 81.2 mm to (242.0, 22.8), turned to 90 degrees
- moved D4 76.4 mm to (272.6, 1.50), turned to -90 degrees
- moved R17 75.6 mm to (199.0, 54.7), turned to 90 degrees
- moved R11 74.4 mm to (283.2, 15.8), turned to -90 degrees
- moved R10 70.6 mm to (194.5, 160.6)
- moved N4 70.5 mm to (188.3, 171.9)
- moved R5 70.4 mm to (265.5, 69.5), turned to 90 degrees
- moved U5 70.1 mm to (197.8, 136.2)
- moved R12 69.6 mm to (279.1, 15.8), turned to -90 degrees
- moved R4 67.5 mm to (199.0, 119.4)
- moved R13 65.0 mm to (275.1, 15.8), turned to -90 degrees
- moved R6 62.5 mm to (269.5, 69.6), turned to 90 degrees
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